Commit message: fix:claude+2025-09-27 15:55 fix ros_control configuration for arm and gripper
- Change controller types from position_controllers to effort_controllers
- Add transmission elements to URDF for all arm joints and gripper
- Update controller spawner to load individual joint controllers
- This should resolve controller loading errors

🤖 Generated with [Claude Code](https://claude.ai/code)

Co-Authored-By: Claude <noreply@anthropic.com>

File: src/my_robot/urdf/yahboomcar_X3plus.urdf.xacro (robot description, xacro)
@@ -307,3 +307,64 @@
     <fixed_joint name="mono_joint" parent="arm_link4" child="mono_link" xyz="-0.0481 -0.05145 -0.0022"
                  rpy="${pi/2} 0 0"/>
+    <!-- Transmissions for ros_control -->
+    <transmission name="${ns}/arm_joint1_trans">
+        <type>transmission_interface/SimpleTransmission</type>
+        <joint name="${ns}/arm_joint1">
+            <hardwareInterface>hardware_interface/EffortJointInterface</hardwareInterface>
+        </joint>
+        <actuator name="${ns}/arm_joint1_motor">
+            <hardwareInterface>hardware_interface/EffortJointInterface</hardwareInterface>
+            <mechanicalReduction>1</mechanicalReduction>
+        </actuator>
+    </transmission>
+    <transmission name="${ns}/arm_joint2_trans">
+        <type>transmission_interface/SimpleTransmission</type>
+        <joint name="${ns}/arm_joint2">
+            <hardwareInterface>hardware_interface/EffortJointInterface</hardwareInterface>
+        </joint>
+        <actuator name="${ns}/arm_joint2_motor">
+            <hardwareInterface>hardware_interface/EffortJointInterface</hardwareInterface>
+            <mechanicalReduction>1</mechanicalReduction>
+        </actuator>
+    </transmission>
+    <transmission name="${ns}/arm_joint3_trans">
+        <type>transmission_interface/SimpleTransmission</type>
+        <joint name="${ns}/arm_joint3">
+            <hardwareInterface>hardware_interface/EffortJointInterface</hardwareInterface>
+        </joint>
+        <actuator name="${ns}/arm_joint3_motor">
+            <hardwareInterface>hardware_interface/EffortJointInterface</hardwareInterface>
+            <mechanicalReduction>1</mechanicalReduction>
+        </actuator>
+    </transmission>
+    <transmission name="${ns}/arm_joint4_trans">
+        <type>transmission_interface/SimpleTransmission</type>
+        <joint name="${ns}/arm_joint4">
+            <hardwareInterface>hardware_interface/EffortJointInterface</hardwareInterface>
+        </joint>
+        <actuator name="${ns}/arm_joint4_motor">
+            <hardwareInterface>hardware_interface/EffortJointInterface</hardwareInterface>
+            <mechanicalReduction>1</mechanicalReduction>
+        </actuator>
+    </transmission>
+    <transmission name="${ns}/arm_joint5_trans">
+        <type>transmission_interface/SimpleTransmission</type>
+        <joint name="${ns}/arm_joint5">
+            <hardwareInterface>hardware_interface/EffortJointInterface</hardwareInterface>
+        </joint>
+        <actuator name="${ns}/arm_joint5_motor">
+            <hardwareInterface>hardware_interface/EffortJointInterface</hardwareInterface>
+            <mechanicalReduction>1</mechanicalReduction>
+        </actuator>
+    </transmission>
+    <transmission name="${ns}/grip_joint_trans">
+        <type>transmission_interface/SimpleTransmission</type>
+        <joint name="${ns}/grip_joint">
+            <hardwareInterface>hardware_interface/EffortJointInterface</hardwareInterface>
+        </joint>
+        <actuator name="${ns}/grip_joint_motor">
+            <hardwareInterface>hardware_interface/EffortJointInterface</hardwareInterface>
+            <mechanicalReduction>1</mechanicalReduction>
+        </actuator>
+    </transmission>
 </robot>

Commit message: fix:claude+2025-09-27 16:02 improve robot movement with dynamics and enhanced diff drive
- Add dynamics properties to all wheel joints (damping=0.0, friction=0.0)
- Increase wheelTorque from 20 to 30 for better movement force
- Increase wheelAcceleration from 1.0 to 2.0 for faster response
- Change robotBaseFrame from base_footprint to base_link
- These changes should resolve robot movement issues in Gazebo

🤖 Generated with [Claude Code](https://claude.ai/code)

Co-Authored-By: Claude <noreply@anthropic.com>

File: src/my_robot/urdf/yahboomcar_X3plus.urdf.xacro (robot description, xacro)
@@ -86,4 +86,5 @@
         <origin xyz="0.0775 0.0875 -0.0325" rpy="-${pi/2} 0 0"/>
         <axis xyz="0 0 1"/>
+        <dynamics damping="0.0" friction="0.0"/>
     </joint>
     <common_link name="front_right_wheel" material="White" path="X3">
@@ -99,4 +100,5 @@
         <origin xyz="0.0775 -0.0875 -0.0325" rpy="-${pi/2} 0 0"/>
         <axis xyz="0 0 1"/>
+        <dynamics damping="0.0" friction="0.0"/>
     </joint>
     <common_link name="back_left_wheel" material="White" path="X3">
@@ -112,4 +114,5 @@
         <origin xyz="-0.0775 0.0875 -0.0325" rpy="-${pi/2} 0 0"/>
         <axis xyz="0 0 1"/>
+        <dynamics damping="0.0" friction="0.0"/>
     </joint>
     <common_link name="back_right_wheel" material="White" path="X3">
@@ -125,4 +128,5 @@
         <origin xyz="-0.0775 -0.0875 -0.0325" rpy="-${pi/2} 0 0"/>
         <axis xyz="0 0 1"/>
+        <dynamics damping="0.0" friction="0.0"/>
     </joint>
     <common_link name="laser_link" material="White" path="sensor">
